File: pcb/koidevboard.kicad_pcb (KiCad board)
At the start: 2 copper layers, 21 x 51 mm, 33 parts, among them J1 USB_C_Receptacle_USB2.0_14P, J2 Conn_01x20, J3 Conn_01x20, J4 Conn_01x03, SW1 SW_Push, U1 RP2040, U2 MCP1700x-300xxTT, U3 W25Q128JVS, Y1 Crystal_GND24

Commit message: silkscreen
Parts:
- added G***: LOGO, Cool Library:glyph, F.Cu at (152.1, 100.5)
- added G***: LOGO, Cool Library:stasis logo, B.Cu at (153.3, 116.6)
- added REF**: KiCad-Logo_5mm_SilkScreen, Symbol:KiCad-Logo_5mm_SilkScreen, B.Cu at (152.4, 121.8)
- added REF**: OSHW-Symbol_6.7x6mm_SilkScreen, Symbol:OSHW-Symbol_6.7x6mm_SilkScreen, B.Cu at (152.4, 80.7)
- renumbered SW1 to SW
Routing:
- net +1V1: track 22.9 -> 22.2 mm
- net GND: vias 29 -> 31
Other:
- board text added: "@cw-urn"
- board text added: "こいでぶ ぼーど"

Commit message: square pads
Routing:
- net GND: track 11.1 -> 13.5 mm, vias 31 -> 32
Changed lines of the file:
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@@
 			(at 0 -1.16 90)
 			(layer "F.SilkS")
+			(hide yes)
 			(effects
 				(font
@@
 			(at 0 -1.16 90)
 			(layer "F.SilkS")
+			(hide yes)
 			(effects
 				(font
@@
 			(at 0 -1.16 90)
 			(layer "F.SilkS")
+			(hide yes)
 			(effects
 				(font
@@
 			(at 0 -1.16 90)
 			(layer "F.SilkS")
+			(hide yes)
 			(effects
 				(font
@@
 			(at 0 -1.16 90)
 			(layer "F.SilkS")
+			(hide yes)
 			(effects
 				(font
@@
 			)
 		)
-		(pad "1" thru_hole rect
+		(pad "1" thru_hole circle
 			(at 0 0 270)
 			(size 1.7 1.7)
@@
 			(pintype "passive")
 		)
-		(pad "2" thru_hole circle
+		(pad "2" thru_hole rect
 			(at 0 -2.54 270)
 			(size 1.7 1.7)
@@
 			)
 		)
-		(pad "1" thru_hole rect
+		(pad "1" thru_hole circle
 			(at 0 0)
 			(size 1.7 1.7)
@@
 			(pintype "passive")
 		)
-		(pad "3" thru_hole circle
+		(pad "3" thru_hole rect
 			(at 0 -5.08)
 			(size 1.7 1.7)
@@
 			(pintype "passive")
 		)
-		(pad "8" thru_hole circle
+		(pad "8" thru_hole rect
 			(at 0 -17.78)
 			(size 1.7 1.7)
@@
 			(pintype "passive")
 		)
-		(pad "13" thru_hole circle
+		(pad "13" thru_hole rect
 			(at 0 -30.48)
 			(size 1.7 1.7)
@@
 			(pintype "passive")
 		)
-		(pad "18" thru_hole circle
+		(pad "18" thru_hole rect
 			(at 0 -43.18)
 			(size 1.7 1.7)
@@
 			)
 		)
-		(pad "1" thru_hole rect
+		(pad "1" thru_hole circle
 			(at 0 0 180)
 			(size 1.7 1.7)
@@
 			(pintype "passive")
 		)
-		(pad "3" thru_hole circle
+		(pad "3" thru_hole rect
 			(at 0 -5.08 180)
 			(size 1.7 1.7)
@@
 			(pintype "passive")
 		)
-		(pad "8" thru_hole circle
+		(pad "8" thru_hole rect
 			(at 0 -17.78 180)
 			(size 1.7 1.7)
@@
 			(pintype "passive")
 		)
-		(pad "13" thru_hole circle
+		(pad "13" thru_hole rect
 			(at 0 -30.48 180)
 			(size 1.7 1.7)
@@
 			(pintype "passive")
 		)
-		(pad "18" thru_hole circle
+		(pad "18" thru_hole rect
 			(at 0 -43.18 180)
 			(size 1.7 1.7)
@@
 	)
 	(segment
+		(start 143.485 107.98)
+		(end 143.58 107.98)
+		(width 0.2)
+		(layer "F.Cu")
+		(net 2)
+	)
+	(segment
 		(start 148.015836 115.5)
 		(end 148.95 115.5)
@@
 	)
 	(segment
+		(start 143.58 107.98)
+		(end 145.2 109.6)
+		(width 0.2)
+		(layer "F.Cu")
+		(net 2)
+	)
+	(segment
 		(start 150.65 113.3)
 		(end 149.789963 114.160037)
@@
 		(size 0.6)
 		(drill 0.3)
+		(layers "F.Cu" "B.Cu")
+		(net 2)
+	)
+	(via
+		(at 145.2 109.6)
+		(size 0.6)
+		(drill 0.3)
